Commit message: adjusting configuration files and others

File: cartographer_ros/urdf/aaucart_2d_IMU.urdf (robot description, URDF)
Before this commit: robot cartographer_aaucart_2d, 3 links, 2 joints
Links:
- added link imu_link; visual box size=0.06 0.04 0.02
Joints:
- added joint imu_link_joint: type fixed, parent base_link, child imu_link, origin xyz=0 0 0
- joint horizontal_laser_link_joint: parent base_link -> imu_link
- joint tilted_laser_link_joint: parent base_link -> imu_link
