Commit message: new adjustments

File: cartographer_ros/urdf/aaucart_2d_odom.urdf (robot description, URDF)
Before this commit: robot cartographer_aaucart_2d, 3 links, 2 joints
Links:
- added link imu_link; visual box size=0.06 0.04 0.02
Joints:
- added joint imu_link_joint: type fixed, parent base_link, child imu_link, origin xyz=0 0 0
- joint horizontal_laser_link_joint: origin xyz=2.04 0 0 -> xyz=1.714 0 -0.154; parent base_link -> imu_link
- joint tilted_laser_link_joint: origin xyz=1.78 0 1.15 rpy=3.141593 0.31 0 -> xyz=1.474 0 0.948 rpy=3.141593 0.31 0; parent base_link -> imu_link
